File: KiCAD/ModularLabPSU/ModularLabPSU.kicad_pcb (KiCad board)
At the start: 2 copper layers, 125 x 80 mm, 145 parts, among them CON1 AVR-ISP-6, IC1 ATMEGA328P-A, J1 USB_MINI_B_OTG, K1 HF115F, P1 CONN_01X04, P2 CONN_01X06, P3 EarthWire, Q1 BC847B, Q2 IRFP044N, Q3 BC847B, Q4 BC847B, Q5 IRFP5210, Q6 IRFP5210, Q7 BC847B, Q8 BC857, Q9 BC847B, U1 LT1639, U10 LM317AT, U11 LM317AT, U12 SCR, U13 LT1716, U14 LTC2050, U2 AD7705BRUZ, U3 AD780BRZ, U4 AD5689, U5 ADUM1201ARZ-RL7, U6 MCP2200, U7 LT1639, U8 LTC2050, U9 LM317HVT, X1 20MHz, X2 12MHz, Y1 2MHz

Commit message: Missing files
Parts:
- added REF**: Symbol_OSHW-Logo_CopperTop, Symbols:Symbol_OSHW-Logo_CopperTop, F.Cu at (139.4, 79.0)
- ?: renamed from REF**; value MountingHole_3.2mm_M3 -> (none)
- moved L1 3.57 mm to (69.4, 68.6)
- moved C14 3.10 mm to (59.1, 84.3)
- moved C15 3.10 mm to (59.1, 86.8)
- moved ? 2.98 mm to (47.0, 47.8)
- moved ? 2.98 mm to (47.0, 120.2)
- moved C3 1.39 mm to (49.8, 109.2)
- moved U3 1.12 mm to (75.5, 92.8)
- moved X2 0.99 mm to (55.9, 74.7)
- moved X1 0.80 mm to (51.2, 113.5)
- moved C4 0.46 mm to (50.0, 105.2)
- moved ? 0.46 mm to (166.9, 47.8)
- moved C13 0.28 mm to (51.6, 75.5), turned to 90 degrees
- moved C12 0.24 mm to (48.3, 75.5), turned to 90 degrees
- renumbered CON1 to ICSP
Routing:
- net VRelay: track 0.00 -> 145.9 mm, vias 0 -> 2
- net +5VD: track 30.8 -> 166.8 mm, vias 0 -> 5
- net Vrect-: track 488.4 -> 577.8 mm, vias 12 -> 37
- net Ioutmon: track 48.3 -> 135.7 mm, vias 3 -> 5
- net +5V: track 154.4 -> 238.9 mm, vias 4 -> 6
- net SetVPlus: track 0.00 -> 82.2 mm
- net VUSB: track 0.00 -> 66.0 mm
- net /DigitalControl/Reset: track 3.96 -> 54.9 mm, vias 0 -> 3
- net Net-(U2-Pad7): track 1.27 -> 49.5 mm, vias 0 -> 2
- net CCMode: track 3.42 -> 51.6 mm, vias 0 -> 2
- net Net-(C6-Pad1): track 0.00 -> 40.9 mm, vias 0 -> 4
- net Net-(IC1-Pad30): track 0.00 -> 33.9 mm
- net Net-(IC1-Pad31): track 0.00 -> 33.2 mm
- net /DigitalControl/SCK: track 39.2 -> 70.5 mm, vias 0 -> 2
- net Net-(U4-Pad3): track 0.00 -> 29.6 mm, vias 0 -> 2
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- added copper zone on B.Cu, net USBGND
- added copper zone on B.Cu, net Vrect-
Other:
- board size 125 x 80 mm -> 128 x 80 mm
- board text added: "Lab PSU V1.2 (c) Runcible Software Pty Ltd 2015"
- board text removed: "Lab PSU V1 (c) Runcible Software Pty Ltd 2015"
