File: KiCAD/ModularLabPSU/VoltageAndCurrentControl.sch (KiCad schematic (older format))
At the start: 50 parts, among them P1 CONN_01X04, P3 EarthWire, Q1 BC847B, Q2 IRFP044N, Q8 BC857, Q9 BC847B, U1 LT1639, U8 LTC2050

Commit message: Started re-design of PCB. Schematic changes from testing first board and started developing new layout
Parts:
- removed R16, R20: 10K, Resistors_SMD:R_0805_HandSoldering, symbol R
- removed R26: 10m, welwyn-oar1:WELWYNOAR1, symbol R
- removed VR3, VR4, VR5, VR6: VR, LittleFuseV275LA20P:V275LA20AP, symbol VR
- added R2: 10m, VC1625:VCS1625, symbol VC1625
- C21: value 100pF -> 4.7pF
- R12, R14, R19, R9: value 4K7 -> 100K*
- R18: value 10K -> 5.1K
Connections:
- net Earth_Protective: now also VR1.2, VR2.2
- net GND: now also R2.I1; no longer R24.2
- net VCC: now also Q8.2 (E); no longer Q8.3 (C)
- net at D5.2 (A), P1.3 (P3): now also R2.I2; no longer U8.3 (+)
- net at R55.2, R56.1: now also Q8.3 (C); no longer Q8.2 (E)
- new net: R2.E2, U8.3 (+)
- new net: R2.E1, R24.2
Other:
- moved on the sheet: P3, R24

Commit message: Missed a couple of stars on precision resistors
Parts:
- R24: value 10R -> 10R*
- R25: value 1K -> 1K*
Changed lines of the file:
@@
 P 3300 6050
 F 0 "R24" V 3380 6050 50  0000 C CNN
-F 1 "10R" V 3300 6050 50  0000 C CNN
+F 1 "10R*" V 3300 6050 50  0000 C CNN
 F 2 "Resistors_SMD:R_0805_HandSoldering" V 3230 6050 30  0001 C CNN
 F 3 "" H 3300 6050 30  0000 C CNN
@@
 P 4650 6150
 F 0 "R25" V 4730 6150 50  0000 C CNN
-F 1 "1K" V 4650 6150 50  0000 C CNN
+F 1 "1K*" V 4650 6150 50  0000 C CNN
 F 2 "Resistors_SMD:R_0805_HandSoldering" V 4580 6150 30  0001 C CNN
 F 3 "" H 4650 6150 30  0000 C CNN
